File: Web/pcb/gate_driver2b.brd (EAGLE design)
At the start: 49.2 x 55.9 mm, 25 parts, among them IC1 HCPL3120, IC2 HCPL3120

Commit message: pcb corrections
Parts:
- moved DC1 1.27 mm to (19.1, 40.6)
- moved DC2 1.27 mm to (19.1, 12.7)
Routing:
- net N$8: track 17.6 -> 21.6 mm
- net N$5: track 16.5 -> 19.1 mm
- net GBOT: track 9.10 -> 7.62 mm
Changed lines of the file:
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@@
 </autorouter>
 <elements>
-<element name="DC1" library="dc-dc-converter" package="NMA" value="" x="17.78" y="40.64" smashed="yes" rot="R90">
-<attribute name="NAME" x="18.796" y="35.687" size="1.27" layer="25" ratio="10" rot="R90"/>
-<attribute name="VALUE" x="21.717" y="38.1" size="1.27" layer="27" ratio="10" rot="R180"/>
-</element>
-<element name="DC2" library="dc-dc-converter" package="NMA" value="" x="17.78" y="12.7" rot="R90"/>
+<element name="DC1" library="dc-dc-converter" package="NMA" value="" x="19.05" y="40.64" smashed="yes" rot="R90">
+<attribute name="NAME" x="20.066" y="35.687" size="1.27" layer="25" ratio="10" rot="R90"/>
+<attribute name="VALUE" x="22.987" y="38.1" size="1.27" layer="27" ratio="10" rot="R180"/>
+</element>
+<element name="DC2" library="dc-dc-converter" package="NMA" value="" x="19.05" y="12.7" rot="R90"/>
 <element name="IC1" library="optocoupler" package="DIL08" value="HCPL3120" x="17.78" y="48.26" rot="R270"/>
 <element name="IC2" library="optocoupler" package="DIL08" value="HCPL3120" x="17.78" y="20.32" smashed="yes" rot="R270">
@@
 <contactref element="C1" pad="2"/>
 <contactref element="IC1" pad="5"/>
-<wire x1="21.59" y1="31.75" x2="21.59" y2="40.64" width="0.6096" layer="16"/>
+<wire x1="21.59" y1="31.75" x2="20.32" y2="31.75" width="0.6096" layer="16"/>
+<wire x1="20.32" y1="31.75" x2="20.32" y2="44.45" width="0.6096" layer="16"/>
+<wire x1="20.32" y1="44.45" x2="21.59" y2="44.45" width="0.6096" layer="16"/>
 <wire x1="21.59" y1="44.45" x2="25.4" y2="44.45" width="0.6096" layer="16"/>
-<wire x1="21.59" y1="40.64" x2="21.59" y2="44.45" width="0.6096" layer="16"/>
 </signal>
 <signal name="N$6">
@@
 <wire x1="22.86" y1="52.07" x2="21.59" y2="52.07" width="0.6096" layer="16"/>
 <polygon width="0.4064" layer="1">
-<vertex x="21.59" y="54.61"/>
+<vertex x="20.32" y="54.61"/>
 <vertex x="31.75" y="54.61"/>
 <vertex x="33.02" y="53.34"/>
@@
 <vertex x="36.83" y="46.99"/>
 <vertex x="36.83" y="30.48"/>
-<vertex x="21.59" y="30.48"/>
+<vertex x="20.32" y="30.48"/>
 </polygon>
 </signal>
@@
 <vertex x="33.02" y="15.24"/>
 <vertex x="35.56" y="17.78"/>
-<vertex x="35.56" y="24.13"/>
-<vertex x="21.59" y="24.13"/>
-<vertex x="21.59" y="1.27"/>
+<vertex x="35.56" y="25.4"/>
+<vertex x="20.32" y="25.4"/>
+<vertex x="20.32" y="1.27"/>
 </polygon>
 </signal>
@@
 <contactref element="C2" pad="2"/>
 <contactref element="IC2" pad="5"/>
-<wire x1="21.59" y1="3.81" x2="21.59" y2="12.7" width="0.6096" layer="16"/>
-<wire x1="21.59" y1="12.7" x2="21.59" y2="16.51" width="0.6096" layer="16"/>
+<wire x1="21.59" y1="3.81" x2="20.32" y2="3.81" width="0.6096" layer="16"/>
+<wire x1="20.32" y1="3.81" x2="20.32" y2="16.51" width="0.6096" layer="16"/>
+<wire x1="20.32" y1="16.51" x2="21.59" y2="16.51" width="0.6096" layer="16"/>
 <wire x1="21.59" y1="16.51" x2="22.86" y2="16.51" width="0.6096" layer="16"/>
-<wire x1="22.86" y1="16.51" x2="25.4" y2="19.05" width="0.6096" layer="16"/>
+<wire x1="22.86" y1="16.51" x2="25.4" y2="16.51" width="0.6096" layer="16"/>
+<wire x1="25.4" y1="16.51" x2="25.4" y2="19.05" width="0.6096" layer="16"/>
 </signal>
 <signal name="N$9">
@@
 <polygon width="0.4064" layer="1">
 <vertex x="1.27" y="54.61"/>
-<vertex x="11.43" y="54.61"/>
-<vertex x="12.7" y="53.34"/>
-<vertex x="12.7" y="43.18"/>
-<vertex x="13.97" y="41.91"/>
-<vertex x="13.97" y="26.67"/>
-<vertex x="12.7" y="25.4"/>
-<vertex x="12.7" y="15.24"/>
-<vertex x="13.97" y="13.97"/>
-<vertex x="13.97" y="2.54"/>
-<vertex x="12.7" y="1.27"/>
+<vertex x="15.24" y="54.61"/>
+<vertex x="15.24" y="1.27"/>
 <vertex x="1.27" y="1.27"/>
 </polygon>
@@
 <contactref element="C3" pad="-"/>
 <polygon width="0.6096" layer="16">
-<vertex x="21.59" y="54.61"/>
+<vertex x="20.32" y="54.61"/>
 <vertex x="31.75" y="54.61"/>
 <vertex x="33.02" y="53.34"/>
@@
 <vertex x="48.26" y="31.75"/>
 <vertex x="46.99" y="30.48"/>
-<vertex x="22.86" y="30.48"/>
-<vertex x="21.59" y="31.75"/>
+<vertex x="20.32" y="30.48"/>
 </polygon>
 </signal>
@@
 <contactref element="R5" pad="2"/>
 <contactref element="D2" pad="C"/>
-<wire x1="31.75" y1="8.89" x2="36.83" y2="8.89" width="1.016" layer="16"/>
-<wire x1="36.83" y1="8.89" x2="35.56" y2="12.7" width="0.6096" layer="16"/>
+<wire x1="31.75" y1="8.89" x2="35.56" y2="8.89" width="1.016" layer="16"/>
+<wire x1="35.56" y1="8.89" x2="35.56" y2="12.7" width="0.6096" layer="16"/>
 <polygon width="0.254" layer="16">
 <vertex x="46.99" y="13.97"/>
@@
 <vertex x="46.99" y="15.24"/>
 <vertex x="48.26" y="16.51"/>
-<vertex x="48.26" y="22.86"/>
-<vertex x="46.99" y="24.13"/>
-<vertex x="21.59" y="24.13"/>
-<vertex x="21.59" y="1.27"/>
+<vertex x="48.26" y="24.13"/>
+<vertex x="46.99" y="25.4"/>
+<vertex x="20.32" y="25.4"/>
+<vertex x="20.32" y="1.27"/>
 </polygon>
 </signal>
@@
 <polygon width="0.4064" layer="16">
 <vertex x="1.27" y="54.61"/>
-<vertex x="11.43" y="54.61"/>
-<vertex x="12.7" y="53.34"/>
-<vertex x="12.7" y="43.18"/>
-<vertex x="13.97" y="41.91"/>
-<vertex x="13.97" y="26.67"/>
-<vertex x="12.7" y="25.4"/>
-<vertex x="12.7" y="15.24"/>
-<vertex x="13.97" y="13.97"/>
-<vertex x="13.97" y="2.54"/>
-<vertex x="12.7" y="1.27"/>
+<vertex x="15.24" y="54.61"/>
+<vertex x="15.24" y="1.27"/>
 <vertex x="1.27" y="1.27"/>
 </polygon>

Commit message: updates
Parts:
- moved D2 1.80 mm to (40.6, 14.0)
- moved R5 1.80 mm to (36.8, 16.5)
- moved D1 1.27 mm to (40.6, 43.2)
- moved R6 1.27 mm to (33.0, 15.2)
- moved C3 1.27 mm to (30.5, 31.8)
- moved C6 1.27 mm to (30.5, 3.81)
- moved R3 1.27 mm to (31.8, 47.0)
Routing:
- net N$9: track 16.3 -> 19.1 mm
- net GBOT: track 7.62 -> 6.35 mm
- net N$10: track 12.7 -> 14.0 mm
- net GTOP: track 5.08 -> 3.81 mm
Other:
- board text added: "Gate Driver V2b"
- board text removed: "Gate Driver V2"
