File: Web/pcb/Hardware v2.0/sensor_voltage.sch (EAGLE design)
At the start: 18 parts, among them IC1 OPA344, IC2 SI8920BCSMD, J1 22-27-2041-04

Commit message: updates
Connections:
- net GND: now also R9.2; no longer JP1.2
- net VCC: now also JP1.2; no longer R9.2
Changed lines of the file:
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@@
 <part name="R6" library="rcl" deviceset="R-EU_" device="0309/12" value="10k"/>
 <part name="R9" library="rcl" deviceset="R-EU_" device="0309/12" value="1k2"/>
-<part name="P+4" library="supply1" library_urn="urn:adsk.eagle:library:371" deviceset="VCC" device=""/>
 <part name="GND1" library="supply1" deviceset="GND" device=""/>
 <part name="R8" library="rcl" deviceset="R-EU_" device="0309/12" value="1k2"/>
@@
 <part name="R3" library="rcl" deviceset="R-EU_" device="0309/12" value="680k"/>
 <part name="VCC2" library="supply1" library_urn="urn:adsk.eagle:library:371" deviceset="VCCIO" device=""/>
-<part name="GND2" library="supply1" deviceset="GND" device=""/>
 <part name="JP1" library="pinhead" deviceset="PINHD-1X2" device=""/>
 <part name="R5" library="rcl" deviceset="R-EU_" device="0309/12" value="10k"/>
@@
 <part name="SUPPLY7" library="supply2" library_urn="urn:adsk.eagle:library:372" deviceset="GND1" device=""/>
 <part name="SUPPLY10" library="supply2" library_urn="urn:adsk.eagle:library:372" deviceset="GND1" device=""/>
+<part name="GND9" library="supply1" deviceset="GND" device=""/>
+<part name="P+4" library="supply1" library_urn="urn:adsk.eagle:library:371" deviceset="VCC" device=""/>
 </parts>
 <sheets>
@@
 <instance part="R6" gate="G$1" x="-71.12" y="0" rot="R180"/>
 <instance part="R9" gate="G$1" x="-53.34" y="-10.16" rot="MR90"/>
-<instance part="P+4" gate="VCC" x="-53.34" y="-2.54"/>
 <instance part="GND1" gate="1" x="-48.26" y="7.62"/>
 <instance part="R8" gate="G$1" x="-48.26" y="15.24" rot="MR90"/>
@@
 <instance part="R3" gate="G$1" x="30.48" y="20.32" rot="R180"/>
 <instance part="VCC2" gate="G$1" x="-5.08" y="25.4" rot="R270"/>
-<instance part="GND2" gate="1" x="-38.1" y="-25.4"/>
 <instance part="JP1" gate="G$1" x="-35.56" y="-17.78"/>
 <instance part="R5" gate="G$1" x="-38.1" y="15.24" rot="R180"/>
@@
 <instance part="SUPPLY7" gate="G$1" x="-5.08" y="15.24" rot="R90"/>
 <instance part="SUPPLY10" gate="G$1" x="-5.08" y="10.16" rot="R90"/>
+<instance part="GND9" gate="1" x="-53.34" y="-2.54" rot="R180"/>
+<instance part="P+4" gate="VCC" x="-38.1" y="-25.4" rot="MR180"/>
 </instances>
 <busses>
@@
 </segment>
 <segment>
-<pinref part="GND2" gate="1" pin="GND"/>
-<pinref part="JP1" gate="G$1" pin="2"/>
-<wire x1="-38.1" y1="-22.86" x2="-38.1" y2="-17.78" width="0.1524" layer="91"/>
-</segment>
-<segment>
 <pinref part="GND7" gate="1" pin="GND"/>
 <pinref part="IC2" gate="G$1" pin="GND"/>
@@
 <pinref part="GND8" gate="1" pin="GND"/>
 <pinref part="J1" gate="-3" pin="S"/>
+</segment>
+<segment>
+<pinref part="R9" gate="G$1" pin="2"/>
+<pinref part="GND9" gate="1" pin="GND"/>
 </segment>
 </net>
@@
 </segment>
 <segment>
-<pinref part="R9" gate="G$1" pin="2"/>
-<pinref part="P+4" gate="VCC" pin="VCC"/>
-</segment>
-<segment>
 <pinref part="R7" gate="G$1" pin="2"/>
 <pinref part="P+5" gate="VCC" pin="VCC"/>
@@
 <pinref part="P+8" gate="VCC" pin="VCC"/>
 </segment>
+<segment>
+<pinref part="JP1" gate="G$1" pin="2"/>
+<pinref part="P+4" gate="VCC" pin="VCC"/>
+<wire x1="-38.1" y1="-22.86" x2="-38.1" y2="-17.78" width="0.1524" layer="91"/>
+</segment>
 </net>

Commit message: updates
Parts:
- removed J1: 22-27-2041-04, con-molex:22-27-2041-04
- removed V1: TME0505S, traco-electronic:TME0505S
- added DC/DC: (no value), dc-dc-converter:MEV3
- added JP2: 22-27-2041-04, con-molex:22-27-2041-04
- C1, C2, C3: value 1uF -> 1µ
- IC1: device OPA344:OPA344 -> SparkFun-AnalogIC:OPA344
- IC2: value SI8920BCSMD -> SI8920; device SI8920BC:SI8920BCSMD -> silabs:SI8920
- R1: value 470 -> 500; device rcl:R-EU_0309/12 -> rcl:R-EU_0207/10
- R2, R3, R4, R5, R6, R7, R8, R9: device rcl:R-EU_0309/12 -> rcl:R-EU_0207/10
Connections:
- removed net N$3 (its old number): IC1.OUT, J1-2.S, R6.2
- removed net N$4 (its old number): IC1.+IN, R4.2, R7.1, R8.2
- removed net N$5 (its old number): J1-1.S, JP1.1, R9.1
- new net N$6: IC1.OUT, JP2-2.S, R6.2
- new net N$8: IC1.+IN, R4.2, R7.2, R8.1
- new net N$9: JP1.1, JP2-1.S, R9.2
- net GND: now also DC/DC.-VIN, JP1.2, JP2-3.S, R8.2; no longer J1-3.S, R8.1, R9.2, V1.-VIN
- net GND1: now also DC/DC.-VOUT; no longer V1.-VOUT
- net VCC: now also DC/DC.+VIN, JP2-4.S, R7.1, R9.1; no longer J1-4.S, JP1.2, R7.2, V1.+VIN
- net VCCIO: now also DC/DC.+VOUT; no longer V1.+VOUT
Other:
- note added: "Read Errata #2!"
- moved on the sheet: C1, C2, C3, IC1, JP1, R1, R2, R3, R4, R5, R6, R7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
