File: Web/pcb/Hardware v2.0/base_board6.brd (EAGLE design)
At the start: 100 x 80 mm, 61 parts, among them IC1 ULN2003AN, IC2 LM2901, IC3 7430N, IC4 LM2596, IC5 MCP2562P, J1 J5MM

Commit message: windows fixes
Parts:
- JP6: device pinhead:1X04 -> pinhead:1X05
- moved JP6 1.27 mm to (31.8, 61.0)
Connections:
- net 3.3V_IN: now also JP6.2; no longer JP6.1
- net GND: now also JP6.5; no longer JP6.4
- net PB10/USART3_TX: now also JP6.3; no longer JP6.2
- net PB11/USART3_RX: now also JP6.4; no longer JP6.3
- net VCC: now also JP6.1
Routing:
- net 3.3V_IN: track 19.9 -> 23.1 mm
Changed lines of the file:
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@@
 <?xml version="1.0" encoding="utf-8"?>
 <!DOCTYPE eagle SYSTEM "eagle.dtd">
-<eagle version="9.1.0">
+<eagle version="6.4">
 <drawing>
 <settings>
 <setting alwaysvectorfont="no"/>
-<setting keepoldvectorfont="yes"/>
 <setting verticaltext="up"/>
 </settings>
@@
 <wire x1="100" y1="80" x2="0" y2="80" width="0" layer="20"/>
 <wire x1="0" y1="80" x2="0" y2="0" width="0" layer="20"/>
-<text x="53.975" y="66.04" size="1.778" layer="25">Motor Inverter Main Board</text>
-<text x="87.63" y="63.5" size="1.778" layer="25">(c) 2017
+<text x="47.625" y="66.675" size="1.6764" layer="25" font="vector" ratio="16">Motor Inverter Main Board</text>
+<text x="85.09" y="63.5" size="1.6764" layer="25" font="vector" ratio="16">(c) 2017
 Johannes
 Huebner</text>
@@
 <param name="dpMaxLengthDifference" value="10mm"/>
 <param name="dpGapFactor" value="2.5"/>
+<param name="checkGrid" value="0"/>
 <param name="checkAngle" value="1"/>
 <param name="checkFont" value="1"/>
 <param name="checkRestrict" value="1"/>
-<param name="checkStop" value="0"/>
-<param name="checkValues" value="0"/>
-<param name="checkNames" value="1"/>
-<param name="checkWireStubs" value="1"/>
-<param name="checkPolygonWidth" value="0"/>
 <param name="useDiameter" value="13"/>
 <param name="maxErrors" value="50"/>
@@
 <pass name="Default">
 <param name="RoutingGrid" value="25mil"/>
-<param name="AutoGrid" value="1"/>
-<param name="Efforts" value="0"/>
-<param name="TopRouterVariant" value="1"/>
 <param name="tpViaShape" value="octagon"/>
 <param name="PrefDir.1" value="|"/>
@@
 </element>
 <element name="C19" library="rcl" package="C025-024X044" value="1µ" x="20.32" y="19.685" rot="R180"/>
-<element name="JP6" library="pinhead" package="1X04" value="" x="30.48" y="60.96" rot="R180"/>
+<element name="JP6" library="pinhead" package="1X05" value="" x="31.75" y="60.96" rot="R180"/>
 <element name="R10" library="rcl" package="0207/10" value="10k" x="75.565" y="22.86" smashed="yes">
 <attribute name="NAME" x="73.787" y="22.479" size="1.27" layer="25" ratio="10"/>
@@
 </element>
 <element name="RN2" library="resistor-net" package="RN-9" value="1.2k" x="68.58" y="39.37" smashed="yes" rot="R270">
+<attribute name="VALUE" x="65.405" y="48.26" size="1.27" layer="27" ratio="10" rot="R270"/>
 <attribute name="NAME" x="67.945" y="54.61" size="1.27" layer="25" ratio="10" rot="R270"/>
-<attribute name="VALUE" x="65.405" y="48.26" size="1.27" layer="27" ratio="10" rot="R270"/>
 </element>
 <element name="IC5" library="SparkFun-DigitalIC" package="DIL08" value="MCP2562P" x="40.005" y="40.005" rot="R270"/>
@@
 <contactref element="C9" pad="2"/>
 <contactref element="C19" pad="2"/>
-<contactref element="JP6" pad="4"/>
 <contactref element="C22" pad="2"/>
 <contactref element="C23" pad="2"/>
@@
 <contactref element="IC1" pad="8"/>
 <contactref element="IC3" pad="7"/>
+<contactref element="JP6" pad="5"/>
 </signal>
 <signal name="VCC">
@@
 <contactref element="IC3" pad="11"/>
 <contactref element="IC3" pad="12"/>
+<contactref element="JP6" pad="1"/>
 </signal>
 <signal name="PA11/CANRX">
@@
 <signal name="PB10/USART3_TX">
 <contactref element="JP2" pad="14"/>
-<contactref element="JP6" pad="2"/>
-<wire x1="31.75" y1="60.96" x2="36.83" y2="55.88" width="0.4064" layer="1"/>
+<contactref element="JP6" pad="3"/>
+<wire x1="36.83" y1="55.88" x2="31.75" y2="60.96" width="0.4064" layer="1"/>
 </signal>
 <signal name="PB11/USART3_RX">
 <contactref element="JP2" pad="15"/>
-<contactref element="JP6" pad="3"/>
-<wire x1="29.21" y1="60.96" x2="29.21" y2="59.69" width="0.4064" layer="1"/>
 <wire x1="29.21" y1="59.69" x2="31.75" y2="57.15" width="0.4064" layer="1"/>
 <wire x1="31.75" y1="57.15" x2="32.385" y2="57.15" width="0.4064" layer="1"/>
@@
 <wire x1="33.02" y1="56.515" x2="33.02" y2="54.61" width="0.4064" layer="1"/>
 <wire x1="33.02" y1="54.61" x2="34.29" y2="53.34" width="0.4064" layer="1"/>
+<contactref element="JP6" pad="4"/>
+<wire x1="29.21" y1="60.96" x2="29.21" y2="59.69" width="0.4064" layer="1"/>
 </signal>
 <signal name="PB12/TIM1_BKIN">
@@
 <signal name="3.3V_IN">
 <contactref element="JP2" pad="5"/>
-<contactref element="JP6" pad="1"/>
-<wire x1="34.29" y1="60.96" x2="44.45" y2="60.96" width="0.4064" layer="16"/>
 <wire x1="46.99" y1="53.34" x2="45.72" y2="54.61" width="0.4064" layer="1"/>
 <wire x1="45.72" y1="54.61" x2="45.72" y2="57.15" width="0.4064" layer="1"/>
@@
 <via x="46.99" y="58.42" extent="1-16" drill="0.6" shape="octagon"/>
 <wire x1="46.99" y1="58.42" x2="44.45" y2="60.96" width="0.4064" layer="16"/>
+<contactref element="JP6" pad="2"/>
+<wire x1="44.45" y1="60.96" x2="39.37" y2="60.96" width="0.4064" layer="16"/>
+<wire x1="39.37" y1="60.96" x2="36.83" y2="58.42" width="0.4064" layer="16"/>
+<wire x1="36.83" y1="58.42" x2="34.925" y2="58.42" width="0.4064" layer="16"/>
+<wire x1="34.925" y1="58.42" x2="34.29" y2="59.055" width="0.4064" layer="16"/>
+<wire x1="34.29" y1="59.055" x2="34.29" y2="60.96" width="0.4064" layer="16"/>
 </signal>
 <signal name="5V_USB">
@@
 </signal>
 </signals>
-<mfgpreviewcolors>
-<mfgpreviewcolor name="soldermaskcolor" color="0xC8008000"/>
-<mfgpreviewcolor name="silkscreencolor" color="0xFFFEFEFE"/>
-<mfgpreviewcolor name="backgroundcolor" color="0xFF282828"/>
-<mfgpreviewcolor name="coppercolor" color="0xFFFFBF00"/>
-<mfgpreviewcolor name="substratecolor" color="0xFF786E46"/>
-</mfgpreviewcolors>
+<errors>
+</errors>
 </board>
 </drawing>
