File: Web/pcb/Hardware v2.0/base_board6.sch (EAGLE design)
At the start: 61 parts, among them IC1 ULN2003AN, IC2 LM2901, IC3 7430N, IC4 LM2596, IC5 MCP2562P, J1 J5MM

Commit message: windows fixes
Parts:
- JP6: device pinhead:PINHD-1X4 -> pinhead:PINHD-1X5
Connections:
- net 3.3V_IN: now also JP6.2; no longer JP6.1
- net GND: now also JP6.5; no longer JP6.4
- net PB10/USART3_TX: now also JP6.3; no longer JP6.2
- net PB11/USART3_RX: now also JP6.4; no longer JP6.3
- net VCC: now also JP6.1
Changed lines of the file:
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@@
 <?xml version="1.0" encoding="utf-8"?>
 <!DOCTYPE eagle SYSTEM "eagle.dtd">
-<eagle version="9.1.0">
+<eagle version="6.4">
 <drawing>
 <settings>
 <setting alwaysvectorfont="no"/>
-<setting keepoldvectorfont="yes"/>
 <setting verticaltext="up"/>
 </settings>
@@
 <part name="C19" library="rcl" deviceset="C-EU" device="025-024X044" value="1µ"/>
 <part name="GND25" library="supply1" deviceset="GND" device=""/>
-<part name="JP6" library="pinhead" deviceset="PINHD-1X4" device=""/>
+<part name="JP6" library="pinhead" deviceset="PINHD-1X5" device=""/>
 <part name="R10" library="rcl" deviceset="R-EU_" device="0207/10" value="10k"/>
 <part name="R11" library="rcl" deviceset="R-EU_" device="0207/10" value="10k"/>
@@
 <part name="P+12" library="supply1" deviceset="VCC" device=""/>
 <part name="P+10" library="supply1" deviceset="VCC" device=""/>
+<part name="GND13" library="supply1" deviceset="GND" device=""/>
+<part name="P+13" library="supply1" deviceset="VCC" device=""/>
 </parts>
 <sheets>
@@
 </instance>
 <instance part="P+10" gate="VCC" x="154.94" y="-7.62" rot="R90"/>
+<instance part="GND13" gate="1" x="-132.08" y="-60.96"/>
+<instance part="P+13" gate="VCC" x="-132.08" y="-35.56"/>
 </instances>
 <busses>
@@
 </segment>
 <segment>
-<wire x1="-132.08" y1="-45.72" x2="-137.16" y2="-45.72" width="0.1524" layer="91"/>
-<label x="-160.02" y="-45.72" size="1.778" layer="95"/>
-<pinref part="JP6" gate="A" pin="2"/>
+<wire x1="-132.08" y1="-48.26" x2="-137.16" y2="-48.26" width="0.1524" layer="91"/>
+<label x="-160.02" y="-48.26" size="1.778" layer="95"/>
+<pinref part="JP6" gate="A" pin="3"/>
 </segment>
 </net>
@@
 </segment>
 <segment>
-<wire x1="-132.08" y1="-48.26" x2="-137.16" y2="-48.26" width="0.1524" layer="91"/>
-<label x="-160.02" y="-48.26" size="1.778" layer="95"/>
-<pinref part="JP6" gate="A" pin="3"/>
+<wire x1="-132.08" y1="-50.8" x2="-137.16" y2="-50.8" width="0.1524" layer="91"/>
+<label x="-160.02" y="-50.8" size="1.778" layer="95"/>
+<pinref part="JP6" gate="A" pin="4"/>
 </segment>
 </net>
@@
 <pinref part="GND25" gate="1" pin="GND"/>
 <pinref part="C19" gate="G$1" pin="2"/>
-</segment>
-<segment>
-<wire x1="-132.08" y1="-50.8" x2="-137.16" y2="-50.8" width="0.1524" layer="91"/>
-<label x="-144.78" y="-50.8" size="1.778" layer="95"/>
-<pinref part="JP6" gate="A" pin="4"/>
 </segment>
 <segment>
@@
 <pinref part="GND11" gate="1" pin="GND"/>
 </segment>
+<segment>
+<pinref part="JP6" gate="A" pin="5"/>
+<pinref part="GND13" gate="1" pin="GND"/>
+<wire x1="-132.08" y1="-58.42" x2="-132.08" y2="-53.34" width="0.1524" layer="91"/>
+</segment>
 </net>
 <net name="VDDA" class="0">
@@
 </segment>
 <segment>
-<wire x1="-132.08" y1="-43.18" x2="-137.16" y2="-43.18" width="0.1524" layer="91"/>
-<label x="-147.32" y="-43.18" size="1.778" layer="95"/>
-<pinref part="JP6" gate="A" pin="1"/>
+<wire x1="-132.08" y1="-45.72" x2="-137.16" y2="-45.72" width="0.1524" layer="91"/>
+<label x="-160.02" y="-45.72" size="1.778" layer="95"/>
+<pinref part="JP6" gate="A" pin="2"/>
 </segment>
 </net>
@@
 <junction x="157.48" y="-7.62"/>
 </segment>
-</net>
+<segment>
+<pinref part="JP6" gate="A" pin="1"/>
+<pinref part="P+13" gate="VCC" pin="VCC"/>
+<wire x1="-132.08" y1="-38.1" x2="-132.08" y2="-43.18" width="0.1524" layer="91"/>
+</segment>
+</net>
