File: Web/pcb/Hardware v2.0/resolver.sch (EAGLE design)
At the start: 17 parts, among them IC1 LM386N-1

Commit message: software updates
Parts:
- added C10: 22n, rcl:C-EU050-024X044
- C9: value 47n -> 22n; device rcl:C-EU025-024X044 -> rcl:C-EU050-024X044
Connections:
- new net N$6: C10.1, C9.1, R6.2
- net N$1: now also C10.2; no longer C9.1, R6.2
