File: Web/pcb/Hardware v3.0/base_board7.sch (EAGLE design)
At the start: 143 parts, among them IC1 LM2596S, IC2A TDA2822D, IC2B LM386M-1, IC3 TJA1040T, IC4 STM32F103RBT6, IC5 MIC2288BML, IC6 ULN2003AD, IC7 LM2901M, IC8 REG1117, IC9A SN74LVC1G10DCKR, IC9B SN74HC10D, Q1 CSM-7X-DU

Commit message: software updates
Parts:
- added L5: (no value), resistor:L-EUTJ3-U1
Connections:
- net N$3: now also L5.1
- net VCC: now also L5.2
Changed lines of the file:
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@@
 <part name="JP16" library="wirepad" library_urn="urn:adsk.eagle:library:412" deviceset="1,6/0,8" device="" package3d_urn="urn:adsk.eagle:package:30830/1"/>
 <part name="JP17" library="wirepad" library_urn="urn:adsk.eagle:library:412" deviceset="1,6/0,8" device="" package3d_urn="urn:adsk.eagle:package:30830/1"/>
+<part name="L5" library="resistor" library_urn="urn:adsk.eagle:library:348" deviceset="L-EU" device="TJ3-U1" package3d_urn="urn:adsk.eagle:package:23496/1"/>
 </parts>
 <sheets>
@@
 <attribute name="VALUE" x="93.98" y="95.25" size="1.778" layer="96" rot="R270"/>
 </instance>
+<instance part="L5" gate="G$1" x="35.56" y="170.18" smashed="yes" rot="R90">
+<attribute name="VALUE" x="39.37" y="173.482" size="1.778" layer="96" rot="R180"/>
+</instance>
 </instances>
 <busses>
@@
 <pinref part="L2" gate="G$1" pin="2"/>
 <junction x="27.94" y="165.1"/>
+<pinref part="L5" gate="G$1" pin="1"/>
+<wire x1="30.48" y1="170.18" x2="27.94" y2="170.18" width="0.1524" layer="91"/>
+<wire x1="27.94" y1="170.18" x2="27.94" y2="165.1" width="0.1524" layer="91"/>
 </segment>
 </net>
@@
 <junction x="53.34" y="165.1"/>
 <wire x1="53.34" y1="165.1" x2="53.34" y2="160.02" width="0.1524" layer="91"/>
-</segment>
-<segment>
+<pinref part="L5" gate="G$1" pin="2"/>
+<wire x1="40.64" y1="170.18" x2="43.18" y2="170.18" width="0.1524" layer="91"/>
+<wire x1="43.18" y1="170.18" x2="43.18" y2="165.1" width="0.1524" layer="91"/>
+</segment>
+<segment>

Commit message: swd over esp progress
Parts:
- L1, L3, L4: device rcl:L-EUL2012C -> rcl:L-EUL3225M

Commit message: some pcb optimizations
Parts:
- added TP1: TPB1,27, testpad:TPB1,27
- ALIVE, PWR: device eagle-ltspice:LED_E -> led:LEDSML0805
Changed lines of the file:
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@@
 <parts>
 <part name="IC4" library="STM32F103RBT6" deviceset="STM32F103RBT6" device=""/>
-<part name="ALIVE" library="eagle-ltspice" library_urn="urn:adsk.eagle:library:217" deviceset="LED_E" device="" package3d_urn="urn:adsk.eagle:package:13319/1" value="LED_0603_GN"/>
+<part name="ALIVE" library="led" library_urn="urn:adsk.eagle:library:259" deviceset="LED" device="SML0805" package3d_urn="urn:adsk.eagle:package:15830/1" value="LED_0603_GN"/>
 <part name="R33" library="rcl" library_urn="urn:adsk.eagle:library:334" deviceset="R-EU_" device="R0603" package3d_urn="urn:adsk.eagle:package:23555/2" value="510"/>
 <part name="VCC1" library="supply1" library_urn="urn:adsk.eagle:library:371" deviceset="VCCIO" device=""/>
@@
 <part name="P+2" library="supply1" library_urn="urn:adsk.eagle:library:371" deviceset="+12V" device=""/>
 <part name="R32" library="rcl" library_urn="urn:adsk.eagle:library:334" deviceset="R-EU_" device="R0603" package3d_urn="urn:adsk.eagle:package:23555/2" value="510"/>
-<part name="PWR" library="eagle-ltspice" library_urn="urn:adsk.eagle:library:217" deviceset="LED_E" device="" package3d_urn="urn:adsk.eagle:package:13319/1" value="LED_0603_RED"/>
+<part name="PWR" library="led" library_urn="urn:adsk.eagle:library:259" deviceset="LED" device="SML0805" package3d_urn="urn:adsk.eagle:package:15830/1" value="LED_0603_RED"/>
 <part name="IC5" library="MIC2288" deviceset="MIC2288BML" device=""/>
 <part name="C23" library="resistor" library_urn="urn:adsk.eagle:library:348" deviceset="C-EU" device="C0603K" package3d_urn="urn:adsk.eagle:package:26200/1" value="1µ"/>
@@
 <part name="JP17" library="wirepad" library_urn="urn:adsk.eagle:library:412" deviceset="1,6/0,8" device="" package3d_urn="urn:adsk.eagle:package:30830/1"/>
 <part name="L5" library="resistor" library_urn="urn:adsk.eagle:library:348" deviceset="L-EU" device="TJ3-U1" package3d_urn="urn:adsk.eagle:package:23496/1"/>
+<part name="TP1" library="testpad" library_urn="urn:adsk.eagle:library:385" deviceset="TP" device="B1,27" package3d_urn="urn:adsk.eagle:package:27944/1" value="TPB1,27"/>
 </parts>
 <sheets>
@@
 <attribute name="VALUE" x="39.37" y="173.482" size="1.778" layer="96" rot="R180"/>
 </instance>
+<instance part="TP1" gate="G$1" x="109.22" y="147.32" smashed="yes">
+<attribute name="NAME" x="107.95" y="148.59" size="1.778" layer="95"/>
+<attribute name="TP_SIGNAL_NAME" x="110.49" y="146.05" size="1.778" layer="97"/>
+</instance>
 </instances>
