File: Web/pcb/Hardware v3.0/usb2can.sch (EAGLE design)
At the start: 48 parts, among them CON1 USB_A_MALESMD, IC1 ADM3053M, IC2 LD1117S33

Commit message: updates
Parts:
- IC1: value ADM3053M -> ADM3053; device ADM3053:ADM3053M -> ADM3053:ADM3053
Other:
- note added: "DFU"
- note added: "MODE"
- note added: "RESET"
